File: adapter.kicad_pcb (KiCad board)
At the start: 2 copper layers, 46.2 x 18.3 mm, 11 parts, among them P1 CONN_01X03, U1 29LV640, U2 LD1117-3.3, U3 SNES_Mask_ROM

Commit message: Routed PCB
Parts:
- U1: value 29LV640 -> TSOP48
Routing:
- net +5V: track 0.00 -> 51.3 mm
- net GND: track 0.00 -> 41.5 mm, vias 0 -> 3
- net +3V3: track 0.00 -> 40.7 mm, vias 0 -> 1
- net /A17: track 0.00 -> 36.4 mm, vias 0 -> 1
- net /OE: track 0.00 -> 30.0 mm, vias 0 -> 1
- net /A19: track 0.00 -> 27.3 mm
- net /A10: track 0.00 -> 18.4 mm
- net /A2: track 0.00 -> 17.1 mm
- net /A16: track 0.00 -> 16.9 mm, vias 0 -> 1
- net /RST: track 0.00 -> 16.7 mm, vias 0 -> 1
- net /A3: track 0.00 -> 16.7 mm, vias 0 -> 1
- net /D3: track 0.00 -> 16.6 mm
- net /A9: track 0.00 -> 16.5 mm, vias 0 -> 1
- net Net-(U1-Pad45): track 0.00 -> 16.1 mm, vias 0 -> 1
- net /A20: track 0.00 -> 15.5 mm, vias 0 -> 1
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